File: Clock Circuit/Clock Circuit.kicad_pcb (KiCad board)
At the start: 2 copper layers, 28 parts, among them SW1 CLK_MAN, SW2 SW_SPDT, U1 4069, U2 NE556, U3 4011

Commit message: Add files via upload
Parts:
- removed /RESET1, RESET1: Conn_01x01_Female, Connector_PinHeader_1.00mm:PinHeader_1x01_P1.00mm_Vertical
- moved R5 78.9 mm to (114.3, 101.6), turned to 90 degrees
- moved D1 76.3 mm to (114.3, 91.4), turned to 90 degrees
- moved SW2 55.3 mm to (123.0, 114.3)
- moved CLOCK1 46.4 mm to (175.3, 114.3)
- moved HLT1 46.4 mm to (170.2, 114.3)
- moved U3 46.0 mm to (162.6, 100.3), turned to 90 degrees
- moved R2 42.0 mm to (116.8, 78.7)
- moved C3 41.0 mm to (137.2, 78.7)
- moved R3 39.2 mm to (147.3, 100.3)
- moved R4 39.2 mm to (152.4, 100.3)
- moved /CLOCK1 38.9 mm to (180.3, 114.3)
- moved C7 38.1 mm to (170.2, 81.3)
- moved SW1 35.7 mm to (133.2, 109.2)
- moved C4 30.7 mm to (145.3, 78.7)
- moved RV1 25.4 mm to (160.0, 78.7)
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Routing:
- net Earth: track 0.00 -> 45.2 mm
- net +5V: track 0.00 -> 41.9 mm
Other:
- board outline added: 101.6 x 40.6 mm

Commit message: Add files via upload
Parts:
- added /CLOCK2: Conn_01x01_Female, Connector_PinHeader_1.00mm:PinHeader_1x01_P1.00mm_Vertical, F.Cu at (179.7, 83.8)
- added CLOCK2: Conn_01x01_Female, Connector_PinHeader_1.00mm:PinHeader_1x01_P1.00mm_Vertical, F.Cu at (179.7, 87.6)
- SW1: value CLK_MAN -> SW_Push_Dual; footprint Button_Switch_THT:SW_PUSH_6mm_H4.3mm -> Button_Switch_THT:SW_TH_Tactile_Omron_B3F-10xx
- moved HLT1 79.5 mm to (90.8, 109.9)
- moved U3 73.8 mm to (88.9, 95.2)
- moved R2 50.0 mm to (157.5, 108.0)
- moved SW1 50.0 mm to (174.3, 80.7), turned to 90 degrees
- moved /CLOCK1 45.3 mm to (135.3, 109.9)
- moved SW2 41.2 mm to (135.3, 75.0), turned to 180 degrees
- moved R5 38.2 mm to (142.2, 75.6), turned to -90 degrees
- moved R1 37.8 mm to (152.4, 95.2), turned to 90 degrees
- moved CLOCK1 37.1 mm to (138.4, 109.9)
- moved RV1 31.9 mm to (171.5, 108.5), turned to 90 degrees
- moved U1 29.7 mm to (123.2, 95.2)
- moved R3 29.6 mm to (176.5, 95.2)
- moved U2 29.6 mm to (156.2, 95.2)
- moved D1 26.7 mm to (139.7, 83.2), turned to 180 degrees
- moved C4 25.9 mm to (170.9, 82.5), turned to 180 degrees
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Connections:
- SW1 pad 2: Earth -> Net-(U2B-TR)
Routing:
- net +5V: track 41.9 -> 187.8 mm, vias 0 -> 1
- net /CLOCK: track 0.00 -> 129.6 mm, vias 0 -> 2
- net CLOCK: track 0.00 -> 91.5 mm, vias 0 -> 2
- net CLOCK_MAN: track 0.00 -> 78.0 mm, vias 0 -> 2
- net Net-(U2A-Q): track 0.00 -> 50.1 mm, vias 0 -> 3
- net Net-(U1-Pad6): track 0.00 -> 49.2 mm
- net SELECT: track 0.00 -> 49.0 mm
- net HLT: track 0.00 -> 48.6 mm
- net CLOCK_AUTO: track 0.00 -> 40.5 mm
- net Net-(U2A-THR): track 0.00 -> 40.4 mm
- net Earth: track 45.2 -> 6.09 mm, vias 0 -> 1
- net Net-(U3-Pad13): track 0.00 -> 37.0 mm
- net Net-(U1-Pad4): track 0.00 -> 36.0 mm, vias 0 -> 1
- net Net-(U2B-TR): track 0.00 -> 32.2 mm
- net Net-(U2A-DIS): track 0.00 -> 17.2 mm
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- added copper zone on B.Cu, net Earth
Other:
- board outline removed
