File: Clock Circuit/Clock Circuit.kicad_sch (KiCad schematic)
At the start: 16 parts, among them U2 NE556

Commit message: Add files via upload
Parts:
- removed /CYCLE_RST1: Conn_01x01_Female, Connector_PinHeader_1.00mm:PinHeader_1x01_P1.00mm_Vertical, symbol Connector:Conn_01x01_Female
- added /CLOCK1, CLOCK1, HLT1: Conn_01x01_Female, Connector_PinHeader_1.00mm:PinHeader_1x01_P1.00mm_Vertical, symbol Connector:Conn_01x01_Female
- added C3: 47nF 25V cerâmico, Capacitor_THT:CP_Radial_D5.0mm_P2.00mm, symbol Device:C
- added C4: 10nF 63V poliester, Capacitor_THT:CP_Radial_D5.0mm_P2.00mm, symbol Device:C
- added D1: LED, LED_THT:LED_D3.0mm, symbol Device:LED
- added R3: 10k, Resistor_THT:R_Axial_DIN0204_L3.6mm_D1.6mm_P7.62mm_Horizontal, symbol Device:R
- added R4: 100k, Resistor_THT:R_Axial_DIN0204_L3.6mm_D1.6mm_P7.62mm_Horizontal, symbol Device:R
- added R5: 470, Resistor_THT:R_Axial_DIN0204_L3.6mm_D1.6mm_P7.62mm_Horizontal, symbol Device:R
- added SW1: CLK_MAN, Button_Switch_THT:SW_PUSH_6mm_H4.3mm, symbol Switch:SW_MEC_5G
- added SW2: SW_SPDT, Button_Switch_THT:SW_CuK_OS102011MA1QN1_SPDT_Angled, symbol Switch:SW_SPDT
- added U1: 4069, Package_DIP:DIP-14_W7.62mm, symbol 4xxx:4069
- added U3: 4011, Package_DIP:DIP-14_W7.62mm, symbol 4xxx:4011
- C1: footprint (none) -> Capacitor_THT:CP_Radial_D5.0mm_P2.00mm
- R1: renamed from R2; footprint (none) -> Resistor_THT:R_Axial_DIN0204_L3.6mm_D1.6mm_P7.62mm_Horizontal
- R2: footprint (none) -> Resistor_THT:R_Axial_DIN0204_L3.6mm_D1.6mm_P7.62mm_Horizontal
- RV1: footprint (none) -> Potentiometer_THT:Potentiometer_ACP_CA9-H5_Horizontal
- U2: footprint (none) -> Package_DIP:DIP-14_W7.62mm
Connections:
- net +5V: now also U2.10 (R), U2.14 (VCC), R3.2, R4.2, SW2.1 (A), U1.14 (VDD), U3.14 (VDD)
- net Earth: now also U2.7 (GND), C3.2, C4.2, R5.1, SW1.1 (A), SW1.2 (A), SW2.3 (C), U1.7 (VSS), U3.7 (VSS)
- net at U2.11 (CV): now also C4.1
- net at U2.12 (THR): now also U2.13 (DIS), C3.1, R4.1
- net at U2.8 (TR): now also R3.1, SW1.3 (B), SW1.4 (B)
- net CLOCK_MAN: now reaches U2.9 (Q)
- net CLOCK_MAN: now also U3.6
- net at U2.5 (Q): now also U1.1
- new net: D1.1 (K), R5.2
- new net: U3.11, U3.8
- new net: U3.12, U3.3
- new net: U3.13, U3.4
- new net: U1.6, U3.9
- new net: U1.11, U1.12
- new net: SW2.2 (B), U1.13
- new net: U1.4, U3.5
- new net CLOCK: CLOCK1.1 (Pin_1), D1.2 (A), U1.8
- new net CLOCK_AUTO: U1.2, U3.1
- new net HLT: HLT1.1 (Pin_1), U1.5
- new net SELECT: U1.10, U1.3, U3.2
- new net /CLOCK: /CLOCK1.1 (Pin_1), U1.9, U3.10
Other:
- company: (none) -> Márcio José Baldo
- title: (none) -> Clock Circuit
- moved on the sheet: C1, C2, R1, R2, RV1, U2A, U2B

Commit message: Add files via upload
Parts:
- removed /RESET1, RESET1: Conn_01x01_Female, Connector_PinHeader_1.00mm:PinHeader_1x01_P1.00mm_Vertical, symbol Connector:Conn_01x01_Female
Changed lines of the file:
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@@
-    )
-  )
-  (global_label "{slash}RESET" (shape input) (at 259.08 22.86 180) (fields_autoplaced)
-    (effects (font (size 1.27 1.27)) (justify right))
-    (property "Intersheetrefs" "${INTERSHEET_REFS}" (at 249.0192 22.86 0)
-      (effects (font (size 1.27 1.27)) (justify right) hide)
-    )
-  )
-  (global_label "RESET" (shape input) (at 259.08 27.94 180) (fields_autoplaced)
-    (effects (font (size 1.27 1.27)) (justify right))
-    (property "Intersheetrefs" "${INTERSHEET_REFS}" (at 250.3497 27.94 0)
-      (effects (font (size 1.27 1.27)) (justify right) hide)
     )
   )
@@
     )
   )
-  (symbol (lib_id "Connector:Conn_01x01_Female") (at 264.16 27.94 0) (mirror x) (unit 1)
-    (in_bom yes) (on_board yes) (dnp no)
-    (property "Reference" "RESET1" (at 269.24 27.94 0)
-      (effects (font (size 1.27 1.27)))
-    )
-    (property "Value" "Conn_01x01_Female" (at 263.525 25.4 0)
-      (effects (font (size 1.27 1.27)))
-    )
-    (property "Footprint" "Connector_PinHeader_1.00mm:PinHeader_1x01_P1.00mm_Vertical" (at 264.16 27.94 0)
-      (effects (font (size 1.27 1.27)) hide)
-    )
-    (property "Datasheet" "~" (at 264.16 27.94 0)
-      (effects (font (size 1.27 1.27)) hide)
-    )
-    (pin "1")
-    (instances
-      (project "Clock Circuit"
-        (path "/4e4768fd-52f0-4853-bca6-f45a0aebc6bd"
-          (reference "RESET1") (unit 1)
-        )
-      )
-      (project "ProgramCounter"
-        (path "/9538e4ed-27e6-4c37-b989-9859dc0d49e8"
-          (reference "RESET1") (unit 1)
-        )
-      )
-    )
-  )
   (symbol (lib_id "Device:C") (at 215.9 77.47 0) (unit 1)
     (in_bom yes) (on_board yes) (dnp no)
@@
         )
       )
-    )
-  )
-  (symbol (lib_id "Connector:Conn_01x01_Female") (at 264.16 22.86 0) (mirror x) (unit 1)
-    (in_bom yes) (on_board yes) (dnp no)
-    (property "Reference" "/RESET1" (at 269.24 22.86 0)
-      (effects (font (size 1.27 1.27)))
-    )
-    (property "Value" "Conn_01x01_Female" (at 263.525 20.32 0)
-      (effects (font (size 1.27 1.27)))
-    )
-    (property "Footprint" "Connector_PinHeader_1.00mm:PinHeader_1x01_P1.00mm_Vertical" (at 264.16 22.86 0)
-      (effects (font (size 1.27 1.27)) hide)
-    )
-    (property "Datasheet" "~" (at 264.16 22.86 0)
-      (effects (font (size 1.27 1.27)) hide)
-    )
-    (pin "1")
-    (instances
-      (project "Clock Circuit"
-        (path "/4e4768fd-52f0-4853-bca6-f45a0aebc6bd"
-          (reference "/RESET1") (unit 1)
-        )
-      )
-      (project "ProgramCounter"
-        (path "/9538e4ed-27e6-4c37-b989-9859dc0d49e8"
-          (reference "/RESET1") (unit 1)
-        )
-      )

Commit message: Add files via upload
Parts:
- removed SW1: CLK_MAN, Button_Switch_THT:SW_PUSH_6mm_H4.3mm, symbol Switch:SW_MEC_5G
- added /CLOCK2, CLOCK2: Conn_01x01_Female, Connector_PinHeader_1.00mm:PinHeader_1x01_P1.00mm_Vertical, symbol Connector:Conn_01x01_Female
- added SW1: SW_Push_Dual, Button_Switch_THT:SW_TH_Tactile_Omron_B3F-10xx, symbol Switch:SW_Push_Dual
Connections:
- net CLOCK: now also CLOCK2.1 (Pin_1)
- net Earth: now also SW1.1, SW1.3
- net /CLOCK: now also /CLOCK2.1 (Pin_1)
- net at R3.1, U2.8 (TR): now also SW1.2, SW1.4
Other:
- moved on the sheet: CLOCK1
